File: tailPCB/tail.sch (EAGLE design)
At the start: 6 parts

Commit message: Add files via upload
Parts:
- removed JP3: (no value), DC_LOAD_AU:PINHD-1X2
- added S1: MOMENTARY-SWITCH-SPST-PTH-6.0MM, SparkFun-Switches:MOMENTARY-SWITCH-SPST-PTH-6.0MM
Connections:
- net 0: now also S1.2; no longer JP3.2
- net N$10: now also S1.1; no longer JP3.1
Changed lines of the file:
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@@
 <part name="R4" library="adafruit" library_urn="urn:adsk.eagle:library:420" deviceset="R-US_" device="0207/10" package3d_urn="urn:adsk.eagle:package:6240597/1" value="1K"/>
 <part name="X_5" library="ngspice-simulation" library_urn="urn:adsk.eagle:library:527439" deviceset="GND" device=""/>
-<part name="JP3" library="DC_LOAD_AU" library_urn="urn:adsk.eagle:library:220454" deviceset="PINHD-1X2" device="" package3d_urn="urn:adsk.eagle:package:220539/2"/>
 <part name="JP2" library="adafruit" library_urn="urn:adsk.eagle:library:420" deviceset="PINHD-1X3" device="" package3d_urn="urn:adsk.eagle:package:6240710/1"/>
 <part name="X_6" library="ngspice-simulation" library_urn="urn:adsk.eagle:library:527439" deviceset="GND" device=""/>
 <part name="X_2" library="ngspice-simulation" library_urn="urn:adsk.eagle:library:527439" deviceset="GND" device=""/>
+<part name="S1" library="SparkFun-Switches" library_urn="urn:adsk.eagle:library:535" deviceset="MOMENTARY-SWITCH-SPST" device="-PTH-6.0MM" package3d_urn="urn:adsk.eagle:package:40163/1"/>
 </parts>
 <sheets>
 <sheet>
 <plain>
-<text x="123.19" y="65.786" size="1.778" layer="95">Drop Button</text>
+<text x="123.19" y="75.946" size="1.778" layer="95">Drop Button</text>
 <text x="60.706" y="105.41" size="1.778" layer="95" rot="R180">+5</text>
 <text x="61.214" y="107.95" size="1.778" layer="95" rot="R180">Ground</text>
@@
 </instance>
 <instance part="X_5" gate="G$1" x="121.92" y="53.34" smashed="yes"/>
-<instance part="JP3" gate="G$1" x="129.54" y="71.12" smashed="yes">
-<attribute name="VALUE" x="123.19" y="66.04" size="1.778" layer="96"/>
-</instance>
 <instance part="JP2" gate="A" x="157.48" y="142.24" smashed="yes" rot="R180">
 <attribute name="VALUE" x="163.83" y="149.86" size="1.778" layer="96" rot="R180"/>
@@
 <instance part="X_6" gate="G$1" x="149.86" y="53.34" smashed="yes"/>
 <instance part="X_2" gate="G$1" x="78.74" y="53.34" smashed="yes"/>
+<instance part="S1" gate="G$1" x="121.92" y="73.66" smashed="yes" rot="R270">
+<attribute name="NAME" x="123.444" y="73.66" size="1.778" layer="95" font="vector" rot="R270" align="bottom-center" display="off"/>
+<attribute name="VALUE" x="121.412" y="73.66" size="1.778" layer="96" font="vector" rot="R270" align="top-center" display="off"/>
+</instance>
 </instances>
 <busses>
@@
 <pinref part="X_4" gate="G$1" pin="0"/>
 <wire x1="106.68" y1="63.5" x2="106.68" y2="53.34" width="0.1524" layer="91"/>
-</segment>
-<segment>
-<pinref part="X_5" gate="G$1" pin="0"/>
-<wire x1="121.92" y1="71.12" x2="121.92" y2="53.34" width="0.1524" layer="91"/>
-<pinref part="JP3" gate="G$1" pin="2"/>
-<wire x1="127" y1="71.12" x2="121.92" y2="71.12" width="0.1524" layer="91"/>
 </segment>
 <segment>
@@
 <junction x="78.74" y="88.9"/>
 </segment>
+<segment>
+<pinref part="S1" gate="G$1" pin="2"/>
+<pinref part="X_5" gate="G$1" pin="0"/>
+<wire x1="121.92" y1="68.58" x2="121.92" y2="53.34" width="0.1524" layer="91"/>
+</segment>
 </net>
 <net name="N$8" class="0">
@@
 <net name="N$10" class="0">
 <segment>
-<pinref part="JP3" gate="G$1" pin="1"/>
-<wire x1="121.92" y1="73.66" x2="127" y2="73.66" width="0.1524" layer="91"/>
-<wire x1="121.92" y1="73.66" x2="121.92" y2="99.06" width="0.1524" layer="91"/>
 <pinref part="W1" gate="G$1" pin="D3"/>
+<wire x1="91.44" y1="99.06" x2="121.92" y2="99.06" width="0.1524" layer="91"/>
+<pinref part="JP1" gate="G$1" pin="7"/>
 <wire x1="121.92" y1="99.06" x2="160.02" y2="99.06" width="0.1524" layer="91"/>
-<pinref part="JP1" gate="G$1" pin="7"/>
 <wire x1="66.04" y1="91.44" x2="91.44" y2="91.44" width="0.1524" layer="91"/>
 <wire x1="91.44" y1="91.44" x2="91.44" y2="99.06" width="0.1524" layer="91"/>
-<wire x1="91.44" y1="99.06" x2="121.92" y2="99.06" width="0.1524" layer="91"/>
+<pinref part="S1" gate="G$1" pin="1"/>
+<wire x1="121.92" y1="78.74" x2="121.92" y2="99.06" width="0.1524" layer="91"/>
 <junction x="121.92" y="99.06"/>
 </segment>
