File: lid schematic/lid.sch (EAGLE design)
At the start: 12 parts, among them Q1 IRL540

Commit message: Add files via upload
Other:
- note added: "D3 (GPIO0)"
- note added: "Wire legend Rx Tx D1 D2 D3 D4 G +5 Yellow Pink Violet Button Closed Open PWM"
- note removed: "D4 (GPIO2)"
Changed lines of the file:
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@@
 <text x="137.414" y="95.758" size="1.778" layer="97">+5V
 from PSU</text>
-<text x="139.446" y="91.948" size="1.27" layer="97">D4 (GPIO2)</text>
+<text x="139.446" y="91.948" size="1.27" layer="97">D3 (GPIO0)</text>
 <text x="109.22" y="66.04" size="1.778" layer="97">Open</text>
 <text x="124.46" y="66.04" size="1.778" layer="97">Closed</text>
@@
 <text x="241.3" y="7.62" size="2.54" layer="94">5</text>
 <text x="99.06" y="66.04" size="1.778" layer="97">Action</text>
+<text x="73.66" y="165.1" size="2.286" layer="97">Wire legend
+Rx  Tx  D1       D2      D3      D4       G +5
+           Yellow  Pink    Violet  Button
+           Closed  Open   PWM</text>
+<wire x1="63.5" y1="180.34" x2="137.16" y2="180.34" width="1.016" layer="97"/>
+<wire x1="137.16" y1="180.34" x2="137.16" y2="160.02" width="1.016" layer="97"/>
+<wire x1="137.16" y1="160.02" x2="63.5" y2="160.02" width="1.016" layer="97"/>
+<wire x1="63.5" y1="160.02" x2="63.5" y2="180.34" width="1.016" layer="97"/>
 </plain>
 <instances>

Commit message: Added LED/FAN GPIO ports
Parts:
- removed JP1: (no value), pinhead:PINHD-1X2
- added JP4: (no value), pinhead:PINHD-1X4
- added USB/PWR: (no value), pinhead:PINHD-1X2
Connections:
- new net N$10: JP4.2, W1.D5
- new net N$11: JP4.3, W1.D6
- net 0: now also JP4.1, JP4.4
- net N$3: now also USB/PWR.2; no longer JP1.2
- net N$8: now also USB/PWR.1; no longer JP1.1
Other:
- note added: "D5"
- note added: "D6"
- note added: "For LED and Fan control"
- note added: "G"
- moved on the sheet: LED1, SV1, W1
