File: Fan/fan control.brd (EAGLE design)
At the start: 49.2 x 16.5 mm, 6 parts, among them CN1 1X4-BIG, CN2 1X4-BIG, Q1 MOSFET-NCHANNEL2N7000

Commit message: Add files via upload
Parts:
- removed CN2: 1X4-BIG, adafruit:1X04-BIG
- added JP1: (no value), pinhead:1X05
- added Q2: MOSFET-NCHANNEL2N7000, digikey:TO-92
- added R3: 1K, adafruit:0207/10
- added R4: 10K, adafruit:0207/10
- added R5, R6: 150R, adafruit:0207/10
- moved Q1 4.02 mm to (27.9, 74.9)
- moved R2 3.81 mm to (17.8, 73.7)
- moved R1 2.54 mm to (17.8, 76.2)
- moved CN1 1.91 mm to (6.99, 68.5)
- moved D1 1.27 mm to (36.8, 73.7), turned to 0 degrees
Connections:
- new net N$5: Q2.2, R3.2, R4.1
- new net N$6: Q2.3, R5.1, R6.1
- new net N$7: CN1.2, R3.1
- new net N$8: JP1.5, R6.2
- new net N$9: JP1.4, R5.2
- net 0: now also Q2.1, R4.2
- net N$1: now also JP1.1, JP1.2; no longer CN2.1
- net N$4: now also JP1.3; no longer CN2.3
Routing:
- net N$5: track 0.00 -> 14.9 mm
- net 0: track 24.8 -> 33.0 mm
- net N$7: track 0.00 -> 6.49 mm
- net N$6: track 0.00 -> 6.35 mm
- net N$1: track 38.5 -> 44.0 mm
- net N$9: track 0.00 -> 3.81 mm
- net N$8: track 0.00 -> 3.81 mm
- net N$4: track 17.0 -> 20.8 mm
- net N$2: track 17.3 -> 14.9 mm
- net N$3: track 7.72 -> 6.89 mm
Other:
- board size 49.2 x 16.5 mm -> 53 x 16.5 mm
- board text added: "(org)"
- board text added: "(violet)"
- board text added: "+"
- board text added: "5V (Red)"
- board text added: "Fan (Blue)"
- board text added: "GND (Black)"
- board text added: "LED (yellow)"
- board text added: "LED+ (Brown)"
- board text added: "LED+ (Tan)"
- board text added: "Motor"
- board text added: "_"
