File: Fan/fan control.sch (EAGLE design)
At the start: 6 parts, among them CN1 1X4-BIG, CN2 1X4-BIG, Q1 MOSFET-NCHANNEL2N7000

Commit message: Add files via upload
Parts:
- removed CN2: 1X4-BIG, adafruit:1X4-BIG
- added JP1: (no value), pinhead:PINHD-1X5
- added Q2: MOSFET-NCHANNEL2N7000, digikey:MOSFET-NCHANNEL2N7000
- added R3: 1K, adafruit:R-US_0207/10
- added R4: 10K, adafruit:R-US_0207/10
- added R5, R6: 150R, adafruit:R-US_0207/10
Connections:
- new net N$5: Q2.G, R3.2, R4.1
- new net N$6: Q2.D, R5.1, R6.1
- new net N$7: CN1.2, R3.1
- new net N$8: JP1.5, R6.2
- new net N$9: JP1.4, R5.2
- net 0: now also Q2.S, R4.2
- net N$1: now also JP1.1, JP1.2; no longer CN2.1
- net N$4: now also JP1.3; no longer CN2.3
Other:
- note added: "2N7000"
- note added: "Fan"
- note added: "LED (Eyes)"
