File: Sounds/DFPlayer/Schematic/DFPlayer-Wemos.sch (EAGLE design)
At the start: 16 parts

Commit message: Add files via upload
Parts:
- removed D1: 1N4004, adafruit:1N4004
- removed LED1: (no value), adafruit:LED5MM
- removed Q1: (no value), adafruit:MOSFET-NGDS_TO220V
- removed R1: 1K, adafruit:R-US_0207/10
- removed S1: MOMENTARY-SWITCH-SPST-PTH-6.0MM, SparkFun-Switches:MOMENTARY-SWITCH-SPST-PTH-6.0MM
- removed SV1: (no value), con-lstb:MA05-1
- added R2: 33K, adafruit:R-US_0207/10
- JP2: value (none) -> Audio Out
- JP3: value (none) -> Power In
- R4: value 1K -> 51K
Connections:
- new net N$10: U$1.RX, W1.D8
- new net N$13: R2.2, R4.2, S4.1, U$1.ADKEY_1, W1.D5
- new net N$6: JP2.2, U$1.DAC_I
- new net N$7: R2.1, S5.1, W1.D6
- new net N$8: R4.1, S6.1
- new net N$9: JP2.3, U$1.DAC_R
- net 0: now also JP2.1, JP3.1, S2.2, S3.2, S4.2, S5.2, S6.2, W1.GND
- net N$2: now also U$1.TX, W1.D7; no longer JP3.1, W1.GND
- net N$4: now also W1.D2
- net N$5: now also W1.D1
Other:
- note added: "+5V"
- note added: "Gnd"
- note added: "Left (tip)"
- note added: "Loop"
- note added: "Play/Pause"
- note added: "Right (ring)"
- note added: "Track 1"
- note removed: "To PSU"
- moved on the sheet: R4, W1

Commit message: Add files via upload
Parts:
- R1: value 51K -> 3K
- renumbered R4 to R1
Connections:
- net N$8: now also W1.D3
Other:
- note added: "Track 2"
- note removed: "Loop"
Changed lines of the file:
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@@
 <part name="FRAME1" library="myParts" deviceset="LETTER_L" device=""/>
 <part name="W1" library="diy-modules" deviceset="WEMOS-D1-MINI" device=""/>
-<part name="R4" library="adafruit" library_urn="urn:adsk.eagle:library:420" deviceset="R-US_" device="0207/10" package3d_urn="urn:adsk.eagle:package:6240597/1" value="51K"/>
+<part name="R1" library="adafruit" library_urn="urn:adsk.eagle:library:420" deviceset="R-US_" device="0207/10" package3d_urn="urn:adsk.eagle:package:6240597/1" value="3K"/>
 <part name="JP2" library="adafruit" library_urn="urn:adsk.eagle:library:420" deviceset="PINHD-1X3" device="" package3d_urn="urn:adsk.eagle:package:6240710/1" value="Audio Out"/>
 <part name="JP3" library="pinhead" library_urn="urn:adsk.eagle:library:325" deviceset="PINHD-1X2" device="" package3d_urn="urn:adsk.eagle:package:22435/2" value="Power In"/>
@@
 <text x="113.284" y="70.104" size="1.778" layer="95" rot="R90">Prev/Vol-</text>
 <text x="123.444" y="70.104" size="1.778" layer="95" rot="R90">Track 1</text>
-<text x="128.524" y="70.104" size="1.778" layer="95" rot="R90">Loop</text>
+<text x="128.524" y="70.104" size="1.778" layer="95" rot="R90">Track 2</text>
 <text x="133.604" y="70.104" size="1.778" layer="95" rot="R90">Play/Pause</text>
 <text x="208.534" y="131.318" size="1.778" layer="95">Gnd</text>
@@
 <attribute name="VALUE" x="93.98" y="106.68" size="1.778" layer="96" rot="R180"/>
 </instance>
-<instance part="R4" gate="G$1" x="129.54" y="95.25" smashed="yes" rot="R90">
+<instance part="R1" gate="G$1" x="129.54" y="95.25" smashed="yes" rot="R90">
 <attribute name="NAME" x="133.1214" y="91.44" size="1.778" layer="95" rot="R90"/>
 <attribute name="VALUE" x="132.842" y="96.52" size="1.778" layer="96" rot="R90"/>
@@
 <segment>
 <pinref part="S6" gate="G$1" pin="1"/>
-<pinref part="R4" gate="G$1" pin="1"/>
-<wire x1="129.54" y1="78.74" x2="129.54" y2="90.17" width="0.1524" layer="91"/>
+<pinref part="R1" gate="G$1" pin="1"/>
+<wire x1="129.54" y1="78.74" x2="129.54" y2="83.82" width="0.1524" layer="91"/>
+<pinref part="W1" gate="G$1" pin="D3"/>
+<wire x1="129.54" y1="83.82" x2="129.54" y2="90.17" width="0.1524" layer="91"/>
+<wire x1="63.5" y1="129.54" x2="53.34" y2="129.54" width="0.1524" layer="91"/>
+<wire x1="53.34" y1="129.54" x2="53.34" y2="83.82" width="0.1524" layer="91"/>
+<wire x1="53.34" y1="83.82" x2="129.54" y2="83.82" width="0.1524" layer="91"/>
+<junction x="129.54" y="83.82"/>
 </segment>
 </net>
@@
 <pinref part="S4" gate="G$1" pin="1"/>
 <wire x1="124.46" y1="104.14" x2="124.46" y2="78.74" width="0.1524" layer="91"/>
-<pinref part="R4" gate="G$1" pin="2"/>
+<pinref part="R1" gate="G$1" pin="2"/>
 <wire x1="129.54" y1="100.33" x2="129.54" y2="104.14" width="0.1524" layer="91"/>
 <pinref part="R2" gate="G$1" pin="2"/>
