File: eggDropPCB/eggDrop.brd (EAGLE design)
At the start: 63.2 x 30.5 mm, 9 parts

Commit message: Add files via upload
Parts:
- added 2N7000: MOSFET-NCHANNEL2N7000, digikey:TO-92
- added JP2: USB pwr, DC_LOAD_AU:1X02
- added JP4: Eyes, DC_LOAD_AU:1X02
- added R2: 10K, adafruit:0207/10
- added R5: 1K, adafruit:0207/10
- JP3: value (none) -> Drop Button
- moved R4 21.3 mm to (40.6, 64.8)
- moved R1 20.7 mm to (40.6, 69.8)
- moved R3 20.4 mm to (40.6, 67.3)
- moved LED1 15.2 mm to (24.1, 73.7)
- moved LED2 15.2 mm to (24.1, 66.0)
- moved LED3 15.2 mm to (24.1, 58.4)
Connections:
- new net N$13: 2N7000.2, R2.1, R5.2
- new net N$14: R5.1, W1.JP1.6
- new net N$2: JP2.2, W1.JP2.8
- new net N$3: 2N7000.3, JP4.2
- net 0: now also 2N7000.1, R2.2
- net N$1: now also JP2.1, JP4.1; no longer W1.JP2.8
Routing:
- net N$13: track 0.00 -> 44.2 mm
- net N$2: track 0.00 -> 39.0 mm
- net N$1: track 69.6 -> 47.2 mm
- net N$14: track 0.00 -> 17.0 mm
- net N$5: track 27.7 -> 12.1 mm
- net N$12: track 22.0 -> 6.61 mm
- net N$3: track 0.00 -> 11.2 mm
- net N$8: track 23.1 -> 12.2 mm
- net N$9: track 5.08 -> 15.8 mm
- net 0: track 87.1 -> 96.7 mm
- net N$6: track 5.08 -> 14.0 mm
- net N$7: track 5.08 -> 10.7 mm
- net N$11: track 47.1 -> 46.0 mm
- net N$10: track 41.8 -> 42.3 mm
Other:
- board text added: "+"
