File: eggDropPCB/eggDrop.sch (EAGLE design)
At the start: 9 parts

Commit message: Add files via upload
Parts:
- added 2N7000: MOSFET-NCHANNEL2N7000, digikey:MOSFET-NCHANNEL2N7000
- added JP2: USB pwr, DC_LOAD_AU:PINHD-1X2
- added JP4: Eyes, DC_LOAD_AU:PINHD-1X2
- added R2: 10K, adafruit:R-US_0207/10
- added R5: 1K, adafruit:R-US_0207/10
- JP3: value (none) -> Drop Button
Connections:
- new net N$13: 2N7000.G, R2.1, R5.2
- new net N$14: R5.1, W1.D7
- new net N$2: JP2.2, W1.5V
- new net N$3: 2N7000.D, JP4.2
- net 0: now also 2N7000.S, R2.2
- net N$1: now also JP2.1, JP4.1; no longer W1.5V
Other:
- note added: "+"
- note added: "_"
- note removed: "Drop Button"
- moved on the sheet: JP1, LED1, LED2, LED3, R1, R3, R4, W1
