File: tail/tail.sch (EAGLE design)
At the start: 6 parts

Commit message: Corrected spelling
On the PC, #include is not case sensitive. It is on Linux.
Parts:
- added JP3: JUMPER-SMT_2_NC_PASTE_NO-SILK, SparkFun-Jumpers:JUMPER-SMT_2_NC_PASTE_NO-SILK
Connections:
- net N$4: now also JP3.2
- net N$6: now also JP3.1
Other:
- note added: "5V Isolation"
- note removed: "Drop Button"
Changed lines of the file:
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@@
 <part name="X_2" library="ngspice-simulation" library_urn="urn:adsk.eagle:library:527439" deviceset="GND" device=""/>
 <part name="S1" library="SparkFun-Switches" library_urn="urn:adsk.eagle:library:535" deviceset="MOMENTARY-SWITCH-SPST" device="-PTH-6.0MM" package3d_urn="urn:adsk.eagle:package:40163/1"/>
+<part name="JP3" library="SparkFun-Jumpers" library_urn="urn:adsk.eagle:library:528" deviceset="JUMPER-SMT_2_NC_PASTE" device="_NO-SILK" package3d_urn="urn:adsk.eagle:package:39283/1" value=""/>
 </parts>
 <sheets>
 <sheet>
 <plain>
-<text x="123.19" y="75.946" size="1.778" layer="95">Drop Button</text>
+<text x="123.19" y="75.946" size="1.778" layer="95">Button</text>
 <text x="60.706" y="105.41" size="1.778" layer="95" rot="R180">+5</text>
 <text x="61.214" y="107.95" size="1.778" layer="95" rot="R180">Ground</text>
@@
 <text x="61.214" y="93.726" size="1.778" layer="95" rot="R180">Button</text>
 <text x="61.214" y="90.17" size="1.778" layer="95" rot="R180">Ground</text>
+<text x="40.894" y="100.33" size="1.778" layer="95" rot="R180">5V Isolation</text>
 </plain>
 <instances>
@@
 <attribute name="VALUE" x="121.412" y="73.66" size="1.778" layer="96" font="vector" rot="R270" align="top-center" display="off"/>
 </instance>
+<instance part="JP3" gate="G$1" x="35.56" y="96.52" smashed="yes"/>
 </instances>
 <busses>
@@
 <wire x1="73.66" y1="96.52" x2="73.66" y2="99.06" width="0.1524" layer="91"/>
 <junction x="73.66" y="99.06"/>
+<pinref part="JP3" gate="G$1" pin="2"/>
+<wire x1="66.04" y1="96.52" x2="40.64" y2="96.52" width="0.1524" layer="91"/>
+<junction x="66.04" y="96.52"/>
 </segment>
 </net>
@@
 <pinref part="W1" gate="G$1" pin="5V"/>
 <wire x1="86.36" y1="106.68" x2="160.02" y2="106.68" width="0.1524" layer="91"/>
+<pinref part="JP3" gate="G$1" pin="1"/>
+<wire x1="30.48" y1="96.52" x2="30.48" y2="93.98" width="0.1524" layer="91"/>
+<wire x1="30.48" y1="93.98" x2="66.04" y2="93.98" width="0.1524" layer="91"/>
+<junction x="66.04" y="93.98"/>
 </segment>
 </net>
